File: schematic/antenna-v1/antenna.kicad_pcb (KiCad board)
At the start: 2 copper layers, 80 x 41 mm, 37 parts, among them J1 CONN_COAXIAL, J2 CONN_COAXIAL, J3 VCC, J4 GND, J5 RJ45, U1 MCP633, U2 MCP633

Commit message: Fix for PCBs: op amps
Parts:
- U1, U2: footprint TO_SOT_Packages_SMD:SOT-23-6 -> Housings_SOIC:SOIC-8_3.9x4.9mm_Pitch1.27mm
- moved C8 5.86 mm to (70.1, 39.3)
- moved R6 5.86 mm to (72.6, 39.3)
- moved U1 3.41 mm to (63.6, 51.7), turned to 0 degrees
- moved U2 2.91 mm to (63.6, 39.7), turned to 0 degrees
Connections:
- U1 pad 1: CH0 -> GND
- U1 pad 2: GND -> CH0
- U1 pad 4: CH0 -> GND
- U1 pad 5: Net-(U1-Pad5) -> GND
- U1 pad 6: +5V -> CH0
- U2 pad 1: CH1 -> GND
- U2 pad 2: GND -> Net-(C3-Pad1)
- U2 pad 4: Net-(C3-Pad1) -> GND
- U2 pad 5: Net-(U2-Pad5) -> GND
- U2 pad 6: +5V -> CH1
Routing:
- net Net-(C3-Pad1): track 19.9 -> 25.3 mm
- net +5V: track 27.4 -> 24.0 mm, vias 6 -> 7
- net CH1: track 36.2 -> 33.0 mm
- net CH0: track 43.7 -> 41.4 mm
- net Net-(C1-Pad1): track 15.1 -> 16.9 mm
- net Net-(C2-Pad1): track 17.6 -> 18.3 mm
Other:
- board text added: "OpenLDS lightning detector antenna, v.1.1"
