File: schematic/v1/gps-timestamper.sch (KiCad schematic (older format))
At the start: 4 parts

Commit message: [PCB] [firmware] Schematics added, GPIO labels added, DAC generated code added
Parts:
- added BZ?: Buzzer, symbol Buzzer
- added C? (x11): 100n, symbol C
- added C?: C, symbol C
- added C? (x2): 100uF, symbol CP
- added C? (x2): 2.2uF, symbol C
- added D?: USBLC6-4SC6, symbol USBLC6-4SC6
- added D? (x8): D, symbol D
- added D?: LCH0, symbol LED
- added D?: LCH1, symbol LED
- added D?: LCH2, symbol LED
- added D?: LCH3, symbol LED
- added D?: LCH7, symbol LED
- added D?: LCH6, symbol LED
- added D?: LCH5, symbol LED
- added D?: LCH4, symbol LED
- added D? (x3): LED, symbol LED
- added J?: USB_B, symbol USB_B
- added J?: SWD, symbol CONN_01X04_MALE
- added J?: GPS, symbol CONN_01X08
- added J?: CONN_01X08, symbol CONN_01X08
- added JP?: Jumper, symbol Jumper
- added R?: 1.5k, symbol R
- added R? (x2): R, symbol R
- added R? (x12): 1k, symbol R
- added R? (x8): 10k, symbol R
- added U?: NCP551, symbol NCP551
- added U? (x8): MCP602, symbol MCP602
- C? (x2): value C -> 20pF
- Y?: value Crystal -> 8MHz
Connections:
- net labels added: +5V, DAC_CH03, DAC_CH47, GPS_MCU_RX, GPS_MCU_TX, LED_ch0, LED_ch1, LED_ch2, LED_ch3, LED_ch4, LED_ch5, LED_ch6, LED_ch7, NRST, PPS_IN, SWCLK, SWDIO, State_ch0, State_ch1, State_ch2, State_ch3, State_ch4, State_ch5, State_ch6, State_ch7, TTL_IN, USB_D+, USB_D-
- wire segments 23 -> 283
Other:
- moved on the sheet: C?, U?, Y?

Commit message: [PCB] [firmware] PCB: version 1 schematic seems normal, firmware: last second period output added
Parts:
- removed C? (x2): 100n, symbol C
- removed D? (x8): D, symbol D
- removed D?: LCH0, symbol LED
- removed D?: LCH1, symbol LED
- removed D?: LCH2, symbol LED
- removed D?: LCH3, symbol LED
- removed D?: LCH7, symbol LED
- removed D?: LCH6, symbol LED
- removed D?: LCH5, symbol LED
- removed D?: LCH4, symbol LED
- removed J?: GPS, symbol CONN_01X08
- removed J?: CONN_01X08, symbol CONN_01X08
- removed R?: R, symbol R
- removed R? (x9): 1k, symbol R
- removed R? (x8): 10k, symbol R
- removed U?: NCP551, symbol NCP551
- removed U? (x8): MCP602, symbol MCP602
- added C11, C12: 100n, Capacitors_SMD:C_0805, symbol C
- added C13: 2.2uF, Capacitors_SMD:C_0805, symbol C
- added C20: 100uF, Capacitors_Tantalum_SMD:CP_Tantalum_Case-B_EIA-3528-21_Wave, symbol CP
- added D1, D2, D3, D5: 1N4148, Diodes_SMD:D_SOD-323, symbol D
- added D10: LED_CH1, LEDs:LED_0805, symbol LED
- added D6: LED_CH0, LEDs:LED_0805, symbol LED
- added J1: GPS, Connect:RJ45_8, symbol RJ45
- added J2: Channel_0, Pin_Headers:Pin_Header_Straight_1x02_Pitch2.54mm, symbol CONN_01X02_FEMALE
- added J3: Channel_1, Pin_Headers:Pin_Header_Straight_1x02_Pitch2.54mm, symbol CONN_01X02_FEMALE
- added L1: Ferrite_Bead, Resistors_SMD:R_0805, symbol Ferrite_Bead
- added R1, R2, R5, R6: 50k, Resistors_SMD:R_0805, symbol R
- added R12, R14: 1k, Resistors_SMD:R_0805, symbol R
- added R13: 470, Resistors_SMD:R_0805, symbol R
- added R3, R4: 10k, Resistors_SMD:R_0805, symbol R
- added R8: 5k, Resistors_SMD:R_0805, symbol R
- added U1, U2, U4, U5, U6, U7: MCP603, TO_SOT_Packages_SMD:SOT-23-6, symbol MCP603
- added U3: APU1206K-33, TO_SOT_Packages_SMD:SOT-223, symbol MCP1826S
- BZ1: renamed from BZ?; footprint (none) -> Buzzers_Beepers:Buzzer_12x9.5RM7.6
- C1, C10, C14, C15, C16, C17, C19, C4, C5, C6, C7, C8, C9: renamed from C?; footprint (none) -> Capacitors_SMD:C_0805
- C18, C3: renamed from C?; footprint (none) -> Capacitors_Tantalum_SMD:CP_Tantalum_Case-B_EIA-3528-21_Wave
- C2: renamed from C?; value C -> 100n; footprint (none) -> Capacitors_SMD:C_0805
- D4: renamed from D?; footprint (none) -> TO_SOT_Packages_SMD:SOT-23-6
- D7, D8, D9: renamed from D?; footprint (none) -> LEDs:LED_0805
- J4: renamed from J?; footprint (none) -> Connect:USB_B
- J5: renamed from J?; footprint (none) -> Pin_Headers:Pin_Header_Straight_1x04_Pitch2.54mm
- JP1: renamed from JP?; footprint (none) -> Connect:GS2
- R10, R11, R7, R9: renamed from R?; footprint (none) -> Resistors_SMD:R_0805
- R15: renamed from R?; value R -> R_buzz; footprint (none) -> Resistors_SMD:R_0805
- U8: renamed from U?; footprint LQFP100 -> Housings_QFP:LQFP-100_14x14mm_Pitch0.5mm
- Y1: renamed from Y?; footprint (none) -> Crystals:Crystal_HC49-U_Vertical
Connections:
- net labels removed: LED_ch0, LED_ch1, LED_ch2, LED_ch3, LED_ch4, LED_ch5, LED_ch6, LED_ch7, State_ch0, State_ch1, State_ch2, State_ch3, State_ch4, State_ch5, State_ch6, State_ch7
- wire segments 283 -> 217

Commit message: [PCB] pcb seems done, silkscreen sims accurate
Parts:
- removed J2: Channel_0, Pin_Headers:Pin_Header_Straight_1x02_Pitch2.54mm, symbol CONN_01X02_FEMALE
- removed J3: Channel_1, Pin_Headers:Pin_Header_Straight_1x02_Pitch2.54mm, symbol CONN_01X02_FEMALE
- added D11: USBLC6-4SC6, TO_SOT_Packages_SMD:SOT-23-6, symbol USBLC6-4SC6
- added J2: Channel0, Connect:SMA_THT_Jack_Straight, symbol CONN_COAXIAL
- added J3: Channel1, Connect:SMA_THT_Jack_Straight, symbol CONN_COAXIAL
Connections:
- wire segments 217 -> 225
Other:
- moved on the sheet: BZ1, C11, C12, C13, C14, C15, C16, C17, D1, D10, D2, D3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

Commit message: [PCB] Design improved. RJ-45 input, buffered PPS output
Parts:
- removed J2: Channel0, Connect:SMA_THT_Jack_Straight, symbol CONN_COAXIAL
- removed J4: USB_B, Connect:USB_B, symbol USB_B
- added C21, C22, C23, C24, C25, C26: 10uF, Capacitors_SMD:C_0805, symbol C
- added J2: Input, Connect:RJ45_8, symbol RJ45
- added J4: USB_OTG, Connect:USB_Micro-B, symbol USB_OTG
- added R16, R17: 1k, Resistors_SMD:R_0805, symbol R
- added U9: 74HC04, SMD_Packages:SOIC-14_N, symbol 74HC04
- J3: value Channel1 -> PPS_OUT
- R8: value 5k -> 10k
Connections:
- net labels added: Ch0_to_amp, Ch1_to_amp, UART_TAG_TX, VCC
- wire segments 225 -> 268
- no-connect marks 0 -> 1
Other:
- note added: "This is for 74HC04\nIt has no special \nVCC and GND pins"
- moved on the sheet: D11, J1

Commit message: [PCB] Active antenna schmatics
Parts:
- U1, U2, U4, U5, U6, U7: value MCP603 -> MCP633
Changed lines of the file:
@@
 P 3950 2350
 F 0 "U6" H 4000 2550 50  0000 C CNN
-F 1 "MCP603" H 4150 2150 50  0000 C CNN
+F 1 "MCP633" H 4150 2150 50  0000 C CNN
 F 2 "TO_SOT_Packages_SMD:SOT-23-6" H 3950 2050 50  0001 L CNN
 F 3 "" H 4000 2550 50  0001 C CNN
@@
 P 1850 1550
 F 0 "U1" H 1900 1750 50  0000 C CNN
-F 1 "MCP603" H 2050 1350 50  0000 C CNN
+F 1 "MCP633" H 2050 1350 50  0000 C CNN
 F 2 "TO_SOT_Packages_SMD:SOT-23-6" H 1850 1250 50  0001 L CNN
 F 3 "" H 1900 1750 50  0001 C CNN
@@
 P 3050 1650
 F 0 "U4" H 3100 1850 50  0000 C CNN
-F 1 "MCP603" H 3250 1450 50  0000 C CNN
+F 1 "MCP633" H 3250 1450 50  0000 C CNN
 F 2 "TO_SOT_Packages_SMD:SOT-23-6" H 3050 1350 50  0001 L CNN
 F 3 "" H 3100 1850 50  0001 C CNN
@@
 P 3950 4000
 F 0 "U7" H 4000 4200 50  0000 C CNN
-F 1 "MCP603" H 4150 3800 50  0000 C CNN
+F 1 "MCP633" H 4150 3800 50  0000 C CNN
 F 2 "TO_SOT_Packages_SMD:SOT-23-6" H 3950 3700 50  0001 L CNN
 F 3 "" H 4000 4200 50  0001 C CNN
@@
 P 1850 3200
 F 0 "U2" H 1900 3400 50  0000 C CNN
-F 1 "MCP603" H 2050 3000 50  0000 C CNN
+F 1 "MCP633" H 2050 3000 50  0000 C CNN
 F 2 "TO_SOT_Packages_SMD:SOT-23-6" H 1850 2900 50  0001 L CNN
 F 3 "" H 1900 3400 50  0001 C CNN
@@
 P 3050 3300
 F 0 "U5" H 3100 3500 50  0000 C CNN
-F 1 "MCP603" H 3250 3100 50  0000 C CNN
+F 1 "MCP633" H 3250 3100 50  0000 C CNN
 F 2 "TO_SOT_Packages_SMD:SOT-23-6" H 3050 3000 50  0001 L CNN
 F 3 "" H 3100 3500 50  0001 C CNN

Commit message: [PCB] Antenna done and input trigger output added for main device
Parts:
- added JP2: Out_select, Pin_Headers:Pin_Header_Straight_1x03_Pitch2.54mm, symbol Jumper_NC_Dual
Connections:
- net PPS_IN: now also JP2.3; no longer U9.1
- net TTL_IN: now also JP2.1
- new net: JP2.2, U9.1
Other:
- moved on the sheet: J3, U9A, U9B, U9C, U9D, U9E, U9F
Changed lines of the file:
@@
 L CONN_COAXIAL J3
 U 1 1 58F96BBE
-P 9550 7850
-F 0 "J3" H 9560 7970 50  0000 C CNN
-F 1 "PPS_OUT" V 9665 7850 50  0000 C CNN
-F 2 "Connect:SMA_THT_Jack_Straight" H 9550 7850 50  0001 C CNN
-F 3 "" H 9550 7850 50  0001 C CNN
-	1    9550 7850
+P 10700 7850
+F 0 "J3" H 10710 7970 50  0000 C CNN
+F 1 "PPS_OUT" V 10815 7850 50  0000 C CNN
+F 2 "Connect:SMA_THT_Jack_Straight" H 10700 7850 50  0001 C CNN
+F 3 "" H 10700 7850 50  0001 C CNN
+	1    10700 7850
 	1    0    0    -1
 $EndComp
@@
 L 74HC04 U9
 U 1 1 58F9E47E
-P 7450 7850
-F 0 "U9" H 7600 7950 50  0000 C CNN
-F 1 "74HC04" H 7650 7750 50  0000 C CNN
-F 2 "SMD_Packages:SOIC-14_N" H 7450 7850 50  0001 C CNN
-F 3 "" H 7450 7850 50  0001 C CNN
-	1    7450 7850
+P 8600 7850
+F 0 "U9" H 8750 7950 50  0000 C CNN
+F 1 "74HC04" H 8800 7750 50  0000 C CNN
+F 2 "SMD_Packages:SOIC-14_N" H 8600 7850 50  0001 C CNN
+F 3 "" H 8600 7850 50  0001 C CNN
+	1    8600 7850
 	1    0    0    -1
 $EndComp
@@
 L 74HC04 U9
 U 2 1 58F9E971
-P 8650 7850
-F 0 "U9" H 8800 7950 50  0000 C CNN
-F 1 "74HC04" H 8850 7750 50  0000 C CNN
-F 2 "SMD_Packages:SOIC-14_N" H 8650 7850 50  0001 C CNN
-F 3 "" H 8650 7850 50  0001 C CNN
-	2    8650 7850
+P 9800 7850
+F 0 "U9" H 9950 7950 50  0000 C CNN
+F 1 "74HC04" H 10000 7750 50  0000 C CNN
+F 2 "SMD_Packages:SOIC-14_N" H 9800 7850 50  0001 C CNN
+F 3 "" H 9800 7850 50  0001 C CNN
+	2    9800 7850
 	1    0    0    -1
 $EndComp
@@
 L 74HC04 U9
 U 3 1 58F9EAF9
-P 8650 8200
-F 0 "U9" H 8800 8300 50  0000 C CNN
-F 1 "74HC04" H 8850 8100 50  0000 C CNN
-F 2 "SMD_Packages:SOIC-14_N" H 8650 8200 50  0001 C CNN
-F 3 "" H 8650 8200 50  0001 C CNN
-	3    8650 8200
+P 9800 8200
+F 0 "U9" H 9950 8300 50  0000 C CNN
+F 1 "74HC04" H 10000 8100 50  0000 C CNN
+F 2 "SMD_Packages:SOIC-14_N" H 9800 8200 50  0001 C CNN
+F 3 "" H 9800 8200 50  0001 C CNN
+	3    9800 8200
 	1    0    0    -1
 $EndComp
@@
 L 74HC04 U9
 U 4 1 58F9EBB2
-P 8650 8550
-F 0 "U9" H 8800 8650 50  0000 C CNN
-F 1 "74HC04" H 8850 8450 50  0000 C CNN
-F 2 "SMD_Packages:SOIC-14_N" H 8650 8550 50  0001 C CNN
-F 3 "" H 8650 8550 50  0001 C CNN
-	4    8650 8550
+P 9800 8550
+F 0 "U9" H 9950 8650 50  0000 C CNN
+F 1 "74HC04" H 10000 8450 50  0000 C CNN
+F 2 "SMD_Packages:SOIC-14_N" H 9800 8550 50  0001 C CNN
+F 3 "" H 9800 8550 50  0001 C CNN
+	4    9800 8550
 	1    0    0    -1
 $EndComp
@@
 L 74HC04 U9
 U 5 1 58F9EC67
-P 8650 8900
-F 0 "U9" H 8800 9000 50  0000 C CNN
-F 1 "74HC04" H 8850 8800 50  0000 C CNN
-F 2 "SMD_Packages:SOIC-14_N" H 8650 8900 50  0001 C CNN
-F 3 "" H 8650 8900 50  0001 C CNN
-	5    8650 8900
+P 9800 8900
+F 0 "U9" H 9950 9000 50  0000 C CNN
+F 1 "74HC04" H 10000 8800 50  0000 C CNN
+F 2 "SMD_Packages:SOIC-14_N" H 9800 8900 50  0001 C CNN
+F 3 "" H 9800 8900 50  0001 C CNN
+	5    9800 8900
 	1    0    0    -1
 $EndComp
@@
 L 74HC04 U9
 U 6 1 58F9ED1A
-P 8650 9250
-F 0 "U9" H 8800 9350 50  0000 C CNN
-F 1 "74HC04" H 8850 9150 50  0000 C CNN
-F 2 "SMD_Packages:SOIC-14_N" H 8650 9250 50  0001 C CNN
-F 3 "" H 8650 9250 50  0001 C CNN
-	6    8650 9250
-	1    0    0    -1
-$EndComp
-Text GLabel 6850 7850 0    60   Input ~ 0
+P 9800 9250
+F 0 "U9" H 9950 9350 50  0000 C CNN
+F 1 "74HC04" H 10000 9150 50  0000 C CNN
+F 2 "SMD_Packages:SOIC-14_N" H 9800 9250 50  0001 C CNN
+F 3 "" H 9800 9250 50  0001 C CNN
+	6    9800 9250
+	1    0    0    -1
+$EndComp
+Text GLabel 7800 7400 0    60   Input ~ 0
 PPS_IN
 $Comp
 L VCC #PWR052
 U 1 1 58FA23E6
-P 7500 8300
-F 0 "#PWR052" H 7500 8150 50  0001 C CNN
-F 1 "VCC" H 7500 8450 50  0000 C CNN
-F 2 "" H 7500 8300 50  0001 C CNN
-F 3 "" H 7500 8300 50  0001 C CNN
-	1    7500 8300
+P 9000 8750
+F 0 "#PWR052" H 9000 8600 50  0001 C CNN
+F 1 "VCC" H 9000 8900 50  0000 C CNN
+F 2 "" H 9000 8750 50  0001 C CNN
+F 3 "" H 9000 8750 50  0001 C CNN
+	1    9000 8750
 	1    0    0    -1
 $EndComp
@@
 L +5V #PWR053
 U 1 1 58FA25C8
-P 7500 8400
-F 0 "#PWR053" H 7500 8250 50  0001 C CNN
-F 1 "+5V" H 7500 8540 50  0000 C CNN
-F 2 "" H 7500 8400 50  0001 C CNN
-F 3 "" H 7500 8400 50  0001 C CNN
-	1    7500 8400
+P 9000 8850
+F 0 "#PWR053" H 9000 8700 50  0001 C CNN
+F 1 "+5V" H 9000 8990 50  0000 C CNN
+F 2 "" H 9000 8850 50  0001 C CNN
+F 3 "" H 9000 8850 50  0001 C CNN
+	1    9000 8850
 	-1   0    0    1
 $EndComp
-Text Notes 6500 8500 0    60   ~ 0
+Text Notes 8000 8950 0    60   ~ 0
 This is for 74HC04\nIt has no special \nVCC and GND pins
 Wire Wire Line
@@
 Connection ~ 3000 6200
 Wire Wire Line
-	9550 8150 9550 8050
+	10700 8150 10700 8050
 Wire Wire Line
 	1700 6850 3400 6850
@@
 	1700 7050 3000 7050
 Wire Wire Line
-	7900 7850 8200 7850
-Wire Wire Line
-	8200 8900 8100 8900
-Wire Wire Line
-	8200 8550 8100 8550
-Connection ~ 8100 8550
-Wire Wire Line
-	8200 8200 8100 8200
-Connection ~ 8100 8200
-Wire Wire Line
-	9100 7850 9400 7850
-Wire Wire Line
-	9200 7850 9200 9250
-Wire Wire Line
-	9200 9250 9100 9250
-Wire Wire Line
-	9100 8900 9200 8900
-Connection ~ 9200 8900
-Wire Wire Line
-	9100 8550 9200 8550
-Connection ~ 9200 8550
-Wire Wire Line
-	9100 8200 9200 8200
-Connection ~ 9200 8200
-Connection ~ 8100 7850
-Wire Wire Line
-	6850 7850 7000 7850
+	9050 7850 9350 7850
+Wire Wire Line
+	9350 8900 9250 8900
+Wire Wire Line
+	9350 8550 9250 8550
+Connection ~ 9250 8550
+Wire Wire Line
+	9350 8200 9250 8200
+Connection ~ 9250 8200
+Wire Wire Line
+	10250 7850 10550 7850
+Wire Wire Line
+	10350 7850 10350 9250
+Wire Wire Line
+	10350 9250 10250 9250
+Wire Wire Line
+	10250 8900 10350 8900
+Connection ~ 10350 8900
+Wire Wire Line
+	10250 8550 10350 8550
+Connection ~ 10350 8550
+Wire Wire Line
+	10250 8200 10350 8200
+Connection ~ 10350 8200
+Connection ~ 9250 7850
+Wire Wire Line
+	8000 7850 8150 7850
 Wire Wire Line
 	5100 7900 5300 7900
-Connection ~ 9200 7850
-Wire Wire Line
-	7500 8300 7500 8400
-Connection ~ 8100 8900
-Wire Wire Line
-	8100 9250 8200 9250
-Wire Wire Line
-	8100 7850 8100 9250
+Connection ~ 10350 7850
+Wire Wire Line
+	9000 8750 9000 8850
+Connection ~ 9250 8900
+Wire Wire Line
+	9250 9250 9350 9250
+Wire Wire Line
+	9250 7850 9250 9250
 $Comp
 L GND #PWR054
 U 1 1 58FA2EC5
-P 9550 8150
-F 0 "#PWR054" H 9550 7900 50  0001 C CNN
-F 1 "GND" H 9550 8000 50  0000 C CNN
-F 2 "" H 9550 8150 50  0001 C CNN
-F 3 "" H 9550 8150 50  0001 C CNN
-	1    9550 8150
+P 10700 8150
+F 0 "#PWR054" H 10700 7900 50  0001 C CNN
+F 1 "GND" H 10700 8000 50  0000 C CNN
+F 2 "" H 10700 8150 50  0001 C CNN
+F 3 "" H 10700 8150 50  0001 C CNN
+	1    10700 8150
 	1    0    0    -1
 $EndComp
@@
 UART_TAG_TX
 Connection ~ 3300 6850
+$Comp
+L Jumper_NC_Dual JP2
+U 1 1 5903395E
+P 7900 7850
+F 0 "JP2" H 7950 7750 50  0000 L CNN
+F 1 "Out_select" H 7900 7950 50  0000 C BNN
+F 2 "Pin_Headers:Pin_Header_Straight_1x03_Pitch2.54mm" H 7900 7850 50  0001 C CNN
+F 3 "" H 7900 7850 50  0001 C CNN
+	1    7900 7850
+	0    -1   -1   0
+$EndComp
+Wire Wire Line
+	7800 7400 7900 7400
+Wire Wire Line
+	7900 7400 7900 7600
+Text GLabel 7800 8250 0    60   Input ~ 0
+TTL_IN
+Wire Wire Line
+	7800 8250 7900 8250
+Wire Wire Line
+	7900 8250 7900 8100
 $EndSCHEMATC

Commit message: Fix for PCBs: op amps
Parts:
- removed U1, U2, U4, U5, U6, U7: MCP633, TO_SOT_Packages_SMD:SOT-23-6, symbol MCP603
- added U1, U2, U4, U5, U6, U7: MCP633, SMD_Packages:SOIC-8-N, symbol CA3130
- U3: value APU1206K-33 -> MCP1826S; footprint TO_SOT_Packages_SMD:SOT-223 -> TO_SOT_Packages_SMD:SOT-223-3_TabPin2
Connections:
- net +3.3VA: now also U1.7 (V+), U2.7 (V+), U4.7 (V+), U5.7 (V+), U6.7 (V+), U7.7 (V+)
- net +3V3: now also U3.3 (VO)
- net +5V: now also U3.1 (VI)
- net DAC_CH03: now also U6.2 (-)
- net DAC_CH47: now also U7.2 (-)
- net GNDA: now also U1.1, U1.3 (+), U1.4 (V-), U1.5, U1.8, U2.1, U2.3 (+), U2.4 (V-), U2.5, U2.8, U4.1, U4.4 (V-), U4.5, U4.8, U5.1, U5.4 (V-), U5.5, U5.8, U6.1, U6.4 (V-), U6.5, U6.8, U7.1, U7.4 (V-), U7.5, U7.8
- net at D3.2 (A), U8.81 (PD0/CAN1_RX/FSMC_D2/FSMC_DA2): now also U6.6
- net at D5.2 (A), U8.82 (PD1/CAN1_TX/FSMC_D3/FSMC_DA3): now also U7.6
- net at R5.1: now also U4.2 (-), U4.6, U6.3 (+)
- net at D1.2 (A): now also U1.6
- net at R1.1, R5.2: now also U1.2 (-)
- net at D1.1 (K), R3.1: now also U4.3 (+)
- net at R6.1: now also U5.2 (-), U5.6, U7.3 (+)
- net at D2.2 (A): now also U2.6
- net at R2.1, R6.2: now also U2.2 (-)
- net at D2.1 (K), R4.1: now also U5.3 (+)
- no-connect marks 1 -> 69

Commit message: GTest external dependency removed, main module schematic upgraded to latest kicad version
Parts:
- BZ1: symbol Buzzer -> gps-timestamper-rescue:Buzzer
- C1, C10, C11, C12, C13, C14, C15, C16, C17, C19, C2, C21, C22, C23, C24, C25, C26, C4, C5, C6, C7, C8, C9: symbol C -> gps-timestamper-rescue:C
- C18, C20, C3: symbol CP -> gps-timestamper-rescue:CP
- D1, D2, D3, D5: symbol D -> gps-timestamper-rescue:D
- D10, D6, D7, D8, D9: symbol LED -> gps-timestamper-rescue:LED
- D11, D4: symbol USBLC6-4SC6 -> usblc6-4sc6:USBLC6-4SC6
- J1, J2: symbol RJ45 -> gps-timestamper-rescue:RJ45
- J3: symbol CONN_COAXIAL -> gps-timestamper-rescue:CONN_COAXIAL
- J4: symbol USB_OTG -> gps-timestamper-rescue:USB_OTG
- J5: symbol CONN_01X04_MALE -> gps-timestamper-rescue:CONN_01X04_MALE
- JP1: symbol Jumper -> gps-timestamper-rescue:Jumper
- JP2: symbol Jumper_NC_Dual -> gps-timestamper-rescue:Jumper_NC_Dual
- L1: symbol Ferrite_Bead -> gps-timestamper-rescue:Ferrite_Bead
- R1, R10, R11, R12, R13, R14, R15, R16, R17, R2, R3, R4, R5, R6, R7, R8, R9: symbol R -> gps-timestamper-rescue:R
- U1, U2, U4, U5, U6, U7: symbol CA3130 -> gps-timestamper-rescue:CA3130
- U3: symbol MCP1826S -> gps-timestamper-rescue:MCP1826S
- U8: symbol STM32F407VGTx -> stm32:STM32F407VGTx
- U9: symbol 74HC04 -> gps-timestamper-rescue:74HC04
- Y1: symbol Crystal -> gps-timestamper-rescue:Crystal
