File: schematic/v1/gps-timestamper.sch (KiCad schematic (older format))
At the start: 73 parts, among them J1 GPS, J2 Input, J3 PPS_OUT, J4 USB_OTG, J5 SWD, U1 MCP633, U2 MCP633, U3 MCP1826S, U4 MCP633, U5 MCP633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

Commit message: New fixed schematics
Parts:
- removed R1, R2, R5, R6: 50k, Resistors_SMD:R_0805, symbol gps-timestamper-rescue:R
- removed R3, R4: 10k, Resistors_SMD:R_0805, symbol gps-timestamper-rescue:R
- added C27, C28: 100n, Capacitors_SMD:C_0805, symbol Device:C
- added D12, D13: 1N4148, Diodes_SMD:D_SOD-323, symbol gps-timestamper-rescue:D
- added R1, R3: 50k, Resistors_SMD:R_0805, symbol Device:R
- added R18, R19, R5, R6: 10k, Resistors_SMD:R_0805, symbol Device:R
- added R2, R4: 47k, Resistors_SMD:R_0805, symbol Device:R
- added U10: MCP633, SMD_Packages:SOIC-8-N, symbol gps-timestamper-rescue:CA3130
Connections:
- net +3.3VA: now also R18.1, U10.7 (V+)
- net Ch0_to_amp: now also U4.3 (+), R2.1
- net Ch1_to_amp: now also U1.3 (+), R1.1
- net GNDA: now also C27.2, C28.2, R19.2, R5.2, R6.2, U10.1, U10.4 (V-), U10.5, U10.8; no longer R16.2, R17.1, U1.3 (+), U2.3 (+)
- net at D1.1 (K): now also D2.1 (K), U7.3 (+), R5.1; no longer U4.3 (+)
- net at D1.2 (A), U1.6: now also U1.2 (-)
- net at U4.2 (-), U4.6: now also D12.2 (A); no longer U6.3 (+)
- net GNDS: now reaches U5.3 (+)
- net GNDS: now also R16.2, R17.1, U2.3 (+), C28.1, U10.2 (-), U10.6; no longer D2.1 (K)
- net at D2.2 (A), U2.6: now also R3.1
- net at U2.2 (-): now also R1.2, R3.2
- new net: D12.1 (K), D13.1 (K), R6.1, U6.3 (+)
- new net: C27.1, R18.2, R19.1, U10.3 (+)
- new net: R2.2, R4.2, U5.2 (-)
- new net: D13.2 (A), R4.1, U5.6
